File: GasSensorShield/GasSensorShield/GasSensorShield.kicad_pcb (KiCad board)
At the start: 2 copper layers, 68.6 x 53.3 mm, 8 parts, among them P1 Power, P2 Analog, P3 Digital, P4 Digital, P5 CONN_01X01, P6 CONN_01X01, P7 CONN_01X01, P8 CONN_01X01

Commit message: Finishing KiCAD & TODO: README.md
Parts:
- added C1: 100n, Capacitor_THT:C_Disc_D4.3mm_W1.9mm_P5.00mm, F.Cu at (126.5, 111.9)
- added C2: 100n, Capacitor_THT:C_Disc_D4.3mm_W1.9mm_P5.00mm, F.Cu at (142.5, 86.4)
- added C3: 1u, Capacitor_THT:C_Disc_D4.3mm_W1.9mm_P5.00mm, F.Cu at (161.0, 95.4)
- added C4: 100n, Capacitor_THT:C_Disc_D4.3mm_W1.9mm_P5.00mm, F.Cu at (152.5, 113.9)
- added J1: Conn_01x03, Connector_PinHeader_2.00mm:PinHeader_1x03_P2.00mm_Vertical, F.Cu at (116.5, 75.9)
- added J2: Conn_01x03, Connector_PinHeader_2.00mm:PinHeader_1x03_P2.00mm_Vertical, F.Cu at (128.5, 81.9)
- added J3: Conn_01x03, Connector_PinHeader_2.00mm:PinHeader_1x03_P2.00mm_Vertical, F.Cu at (114.5, 99.4)
- added R1: 10K, Resistor_THT:R_Axial_DIN0207_L6.3mm_D2.5mm_P10.16mm_Horizontal, F.Cu at (126.5, 96.4)
- added R2: 100k, Resistor_THT:R_Axial_DIN0207_L6.3mm_D2.5mm_P10.16mm_Horizontal, F.Cu at (131.5, 96.4)
- added R3: 1k, Resistor_THT:R_Axial_DIN0207_L6.3mm_D2.5mm_P10.16mm_Horizontal, F.Cu at (139.5, 98.9)
- added R4: 100k, Resistor_THT:R_Axial_DIN0207_L6.3mm_D2.5mm_P10.16mm_Horizontal, F.Cu at (160.0, 98.9)
- added R5: 1k, Resistor_THT:R_Axial_DIN0207_L6.3mm_D2.5mm_P10.16mm_Horizontal, F.Cu at (161.5, 103.4)
- added U1: RN2483_Breakout, Mes_empreintes:Module_RN2483_Breakout, F.Cu at (177.0, 95.4)
- added U2: GasSensor, Package_TO_SOT_THT:TO-5-10, F.Cu at (116.0, 114.4)
- added U3: LTC1050CN, eec:Linear_Technology-LTC1050CN-Manufacturer_Recommended, F.Cu at (151.0, 98.9)
Connections:
- P2 pad 1: /A0 -> ADC
- P3 pad 6: /12(MISO) -> /RST
- P3 pad 7: /11(**/MOSI) -> /RX
- P3 pad 8: /10(**/SS) -> /TX
Routing:
- net GND: track 0.00 -> 136.1 mm, vias 0 -> 1
- net +5V: track 0.00 -> 128.6 mm, vias 0 -> 1
- net /A2: track 0.00 -> 57.6 mm, vias 0 -> 2
- net /GSLeft_in: track 0.00 -> 51.1 mm
- net /RST: track 0.00 -> 49.2 mm
- net Net-(C3-Pad1): track 0.00 -> 46.4 mm, vias 0 -> 2
- net /RX: track 0.00 -> 41.7 mm
- net /GSLeft_out: track 0.00 -> 39.8 mm
- net +3V3: track 0.00 -> 38.6 mm, vias 0 -> 1
- net Net-(C1-Pad1): track 0.00 -> 38.3 mm
- net /TX: track 0.00 -> 37.6 mm
- net /GSRight_in: track 0.00 -> 36.4 mm, vias 0 -> 1
- net /GSRight_out: track 0.00 -> 33.8 mm
- net Net-(C3-Pad2): track 0.00 -> 24.1 mm
- net ADC: track 0.00 -> 19.6 mm
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Other:
- net class Default: clearance 0.2 -> 0.5; trace_width 0.25 -> 0.5; via_dia 0.6 -> 1.8; via_drill 0.4 -> 0.8
- rule trace_clearance: 0.2 -> 0.5
- rule trace_min: 0.2 -> 0.5
- rule via_min_size: 0.4 -> 0.8
