File: GasSensorShield/GasSensorShield/GasSensorShield.sch (KiCad schematic (older format))
At the start: 23 parts, among them J1 Conn_01x03, J2 Conn_01x03, J3 Conn_01x03, P1 Power, P2 Analog, P3 Digital, P4 Digital, P5 CONN_01X01, P6 CONN_01X01, P7 CONN_01X01, P8 CONN_01X01, U1 RN2483_Breakout, U2 GasSensor, U3 LTC1050CN

Commit message: Finishing KiCAD & TODO: README.md
Parts:
- J1, J2, J3: footprint (none) -> Connector_PinHeader_2.00mm:PinHeader_1x03_P2.00mm_Vertical
- U1: footprint (none) -> Mes_empreintes:Module_RN2483_Breakout
- U2: footprint (none) -> Package_TO_SOT_THT:TO-5-10
- U3: footprint Linear_Technology-LTC1050CN-* -> eec:Linear_Technology-LTC1050CN-Manufacturer_Recommended
Changed lines of the file:
@@
 F 0 "U3" H 5094 4196 50  0000 L CNN
 F 1 "LTC1050CN" H 5094 4105 50  0000 L CNN
-F 2 "Linear_Technology-LTC1050CN-*" H 4350 4750 50  0001 L CNN
+F 2 "eec:Linear_Technology-LTC1050CN-Manufacturer_Recommended" H 4350 4750 50  0001 L CNN
 F 3 "http://cds.linear.com/docs/en/datasheet/1050fb.pdf" H 4350 4850 50  0001 L CNN
 F 4 "1" H 4350 4950 50  0001 L CNN "Channels "
@@
 F 0 "U2" H 1725 2515 50  0000 C CNN
 F 1 "GasSensor" H 1725 2424 50  0000 C CNN
-F 2 "" H 1550 2500 50  0001 C CNN
+F 2 "Package_TO_SOT_THT:TO-5-10" H 1550 2500 50  0001 C CNN
 F 3 "" H 1550 2500 50  0001 C CNN
 	1    1550 2500
@@
 F 0 "U1" H 1528 1663 50  0000 L CNN
 F 1 "RN2483_Breakout" H 1528 1572 50  0000 L CNN
-F 2 "" H 1050 1800 50  0001 C CNN
+F 2 "Mes_empreintes:Module_RN2483_Breakout" H 1050 1800 50  0001 C CNN
 F 3 "" H 1050 1800 50  0001 C CNN
 	1    1050 1800
@@
 F 0 "J1" H 3130 1342 50  0000 L CNN
 F 1 "Conn_01x03" H 3130 1251 50  0000 L CNN
-F 2 "" H 3050 1300 50  0001 C CNN
+F 2 "Connector_PinHeader_2.00mm:PinHeader_1x03_P2.00mm_Vertical" H 3050 1300 50  0001 C CNN
 F 3 "~" H 3050 1300 50  0001 C CNN
 	1    3050 1300
@@
 F 0 "J2" H 4530 1342 50  0000 L CNN
 F 1 "Conn_01x03" H 4530 1251 50  0000 L CNN
-F 2 "" H 4450 1300 50  0001 C CNN
+F 2 "Connector_PinHeader_2.00mm:PinHeader_1x03_P2.00mm_Vertical" H 4450 1300 50  0001 C CNN
 F 3 "~" H 4450 1300 50  0001 C CNN
 	1    4450 1300
@@
 F 0 "J3" H 5830 1342 50  0000 L CNN
 F 1 "Conn_01x03" H 5830 1251 50  0000 L CNN
-F 2 "" H 5750 1300 50  0001 C CNN
+F 2 "Connector_PinHeader_2.00mm:PinHeader_1x03_P2.00mm_Vertical" H 5750 1300 50  0001 C CNN
 F 3 "~" H 5750 1300 50  0001 C CNN
 	1    5750 1300
